File: electro/combat_2.0/motors.kicad_sch (KiCad schematic)
At the start: 9 parts, among them J10 Conn_01x03_Pin, J11 Conn_01x03_Pin, U3 TB6612FNG

Commit message: almost ready pcb
Parts:
- removed C4, C8: 10uF, Capacitor_SMD:CP_Elec_4x5.4, symbol Device:C_Polarized_Small
- C11: renamed from C5; value 0.1uF -> 22uF; footprint Capacitor_SMD:C_1206_3216Metric_Pad1.33x1.80mm_HandSolder -> Capacitor_SMD:C_0805_2012Metric_Pad1.18x1.45mm_HandSolder
- C12: renamed from C6; footprint Capacitor_SMD:C_1206_3216Metric_Pad1.33x1.80mm_HandSolder -> Capacitor_SMD:C_0805_2012Metric_Pad1.18x1.45mm_HandSolder
- C13: renamed from C7; footprint Capacitor_SMD:C_1206_3216Metric_Pad1.33x1.80mm_HandSolder -> Capacitor_SMD:C_0805_2012Metric_Pad1.18x1.45mm_HandSolder
- C9: renamed from C3; value 0.1uF -> 22uF; footprint Capacitor_SMD:C_1206_3216Metric_Pad1.33x1.80mm_HandSolder -> Capacitor_SMD:C_0805_2012Metric_Pad1.18x1.45mm_HandSolder
- J4: renamed from J11; footprint Connector_JST:JST_GH_SM02B-GHS-TB_1x02-1MP_P1.25mm_Horizontal -> Connector_Molex:Molex_PicoBlade_53398-0271_1x02-1MP_P1.25mm_Vertical
- J5: renamed from J10; footprint Connector_JST:JST_GH_SM02B-GHS-TB_1x02-1MP_P1.25mm_Horizontal -> Connector_Molex:Molex_PicoBlade_53398-0271_1x02-1MP_P1.25mm_Vertical
Changed lines of the file:
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@@
   (junction (at 114.3 33.02) (diameter 0) (color 0 0 0 0)
   )
-  (junction (at 68.58 43.18) (diameter 0) (color 0 0 0 0)
-  )
   (junction (at 99.06 33.02) (diameter 0) (color 0 0 0 0)
   )
   (junction (at 124.46 50.8) (diameter 0) (color 0 0 0 0)
   )
-  (junction (at 123.19 33.02) (diameter 0) (color 0 0 0 0)
-  )
   (junction (at 124.46 55.88) (diameter 0) (color 0 0 0 0)
   )
@@
   (junction (at 120.65 33.02) (diameter 0) (color 0 0 0 0)
   )
-  (junction (at 133.35 40.64) (diameter 0) (color 0 0 0 0)
-  )
   (junction (at 111.76 33.02) (diameter 0) (color 0 0 0 0)
   )
-  (junction (at 81.28 33.02) (diameter 0) (color 0 0 0 0)
-  )
   (junction (at 109.22 88.9) (diameter 0) (color 0 0 0 0)
   )
@@
     (stroke (width 0) (type default))
   )
-  (wire (pts (xy 68.58 43.18) (xy 81.28 43.18))
-    (stroke (width 0) (type default))
-  )
   (wire (pts (xy 124.46 68.58) (xy 140.97 68.58))
     (stroke (width 0) (type default))
@@
     (stroke (width 0) (type default))
   )
-  (wire (pts (xy 81.28 33.02) (xy 68.58 33.02))
-    (stroke (width 0) (type default))
-  )
   (wire (pts (xy 121.92 50.8) (xy 124.46 50.8))
     (stroke (width 0) (type default))
@@
     (stroke (width 0) (type default))
   )
-  (wire (pts (xy 81.28 33.02) (xy 81.28 35.56))
-    (stroke (width 0) (type default))
-  )
-  (wire (pts (xy 133.35 33.02) (xy 133.35 34.29))
-    (stroke (width 0) (type default))
-  )
-  (wire (pts (xy 68.58 40.64) (xy 68.58 43.18))
-    (stroke (width 0) (type default))
-  )
-  (wire (pts (xy 123.19 33.02) (xy 133.35 33.02))
-    (stroke (width 0) (type default))
-  )
   (wire (pts (xy 121.92 63.5) (xy 124.46 63.5))
     (stroke (width 0) (type default))
@@
     (stroke (width 0) (type default))
   )
-  (wire (pts (xy 81.28 43.18) (xy 81.28 40.64))
-    (stroke (width 0) (type default))
-  )
-  (wire (pts (xy 99.06 33.02) (xy 81.28 33.02))
+  (wire (pts (xy 68.58 33.02) (xy 99.06 33.02))
     (stroke (width 0) (type default))
   )
@@
     (stroke (width 0) (type default))
   )
-  (wire (pts (xy 68.58 46.99) (xy 68.58 43.18))
+  (wire (pts (xy 68.58 40.64) (xy 68.58 46.99))
     (stroke (width 0) (type default))
   )
@@
     (stroke (width 0) (type default))
   )
-  (wire (pts (xy 133.35 40.64) (xy 133.35 39.37))
-    (stroke (width 0) (type default))
-  )
   (wire (pts (xy 120.65 39.37) (xy 120.65 40.64))
     (stroke (width 0) (type default))
@@
     (effects (font (size 1.27 1.27)) (justify right))
   )
-  (symbol (lib_id "Device:C_Polarized_Small") (at 81.28 38.1 0) (unit 1)
-    (in_bom yes) (on_board yes) (dnp no) (fields_autoplaced)
-    (property "Reference" "C4" (at 83.82 36.2838 0)
-      (effects (font (size 1.27 1.27)) (justify left))
-    )
-    (property "Value" "10uF" (at 83.82 38.8238 0)
-      (effects (font (size 1.27 1.27)) (justify left))
-    )
-    (property "Footprint" "Capacitor_SMD:CP_Elec_4x5.4" (at 81.28 38.1 0)
-      (effects (font (size 1.27 1.27)) hide)
-    )
-    (property "Datasheet" "~" (at 81.28 38.1 0)
-      (effects (font (size 1.27 1.27)) hide)
-    )
-    (pin "1")
-    (pin "2")
-    (instances
-      (project "combat_2.0"
-        (path "/518cdd36-e3d2-496e-a534-90a14dea15b3/75a6c3bc-fc0f-431f-8cec-1b3bc24c24b9"
-          (reference "C4") (unit 1)
-        )
-      )
-    )
-  )
   (symbol (lib_id "Device:C_Small") (at 120.65 36.83 0) (unit 1)
     (in_bom yes) (on_board yes) (dnp no) (fields_autoplaced)
-    (property "Reference" "C5" (at 123.19 35.5662 0)
-      (effects (font (size 1.27 1.27)) (justify left))
-    )
-    (property "Value" "0.1uF" (at 123.19 38.1062 0)
-      (effects (font (size 1.27 1.27)) (justify left))
-    )
-    (property "Footprint" "Capacitor_SMD:C_1206_3216Metric_Pad1.33x1.80mm_HandSolder" (at 120.65 36.83 0)
+    (property "Reference" "C11" (at 123.19 35.5662 0)
+      (effects (font (size 1.27 1.27)) (justify left))
+    )
+    (property "Value" "22uF" (at 123.19 38.1062 0)
+      (effects (font (size 1.27 1.27)) (justify left))
+    )
+    (property "Footprint" "Capacitor_SMD:C_0805_2012Metric_Pad1.18x1.45mm_HandSolder" (at 120.65 36.83 0)
       (effects (font (size 1.27 1.27)) hide)
     )
@@
       (project "combat_2.0"
         (path "/518cdd36-e3d2-496e-a534-90a14dea15b3/75a6c3bc-fc0f-431f-8cec-1b3bc24c24b9"
-          (reference "C5") (unit 1)
+          (reference "C11") (unit 1)
         )
       )
@@
     )
   )
-  (symbol (lib_id "Device:C_Polarized_Small") (at 133.35 36.83 0) (unit 1)
-    (in_bom yes) (on_board yes) (dnp no) (fields_autoplaced)
-    (property "Reference" "C8" (at 135.89 35.0138 0)
-      (effects (font (size 1.27 1.27)) (justify left))
-    )
-    (property "Value" "10uF" (at 135.89 37.5538 0)
-      (effects (font (size 1.27 1.27)) (justify left))
-    )
-    (property "Footprint" "Capacitor_SMD:CP_Elec_4x5.4" (at 133.35 36.83 0)
-      (effects (font (size 1.27 1.27)) hide)
-    )
-    (property "Datasheet" "~" (at 133.35 36.83 0)
-      (effects (font (size 1.27 1.27)) hide)
-    )
-    (pin "1")
-    (pin "2")
-    (instances
-      (project "combat_2.0"
-        (path "/518cdd36-e3d2-496e-a534-90a14dea15b3/75a6c3bc-fc0f-431f-8cec-1b3bc24c24b9"
-          (reference "C8") (unit 1)
-        )
-      )
-    )
-  )
   (symbol (lib_id "Device:C_Small") (at 68.58 38.1 0) (unit 1)
     (in_bom yes) (on_board yes) (dnp no) (fields_autoplaced)
-    (property "Reference" "C3" (at 71.12 36.8362 0)
-      (effects (font (size 1.27 1.27)) (justify left))
-    )
-    (property "Value" "0.1uF" (at 71.12 39.3762 0)
-      (effects (font (size 1.27 1.27)) (justify left))
-    )
-    (property "Footprint" "Capacitor_SMD:C_1206_3216Metric_Pad1.33x1.80mm_HandSolder" (at 68.58 38.1 0)
+    (property "Reference" "C9" (at 71.12 36.8362 0)
+      (effects (font (size 1.27 1.27)) (justify left))
+    )
+    (property "Value" "22uF" (at 71.12 39.3762 0)
+      (effects (font (size 1.27 1.27)) (justify left))
+    )
+    (property "Footprint" "Capacitor_SMD:C_0805_2012Metric_Pad1.18x1.45mm_HandSolder" (at 68.58 38.1 0)
       (effects (font (size 1.27 1.27)) hide)
     )
@@
       (project "combat_2.0"
         (path "/518cdd36-e3d2-496e-a534-90a14dea15b3/75a6c3bc-fc0f-431f-8cec-1b3bc24c24b9"
-          (reference "C3") (unit 1)
+          (reference "C9") (unit 1)
         )
       )
@@
   (symbol (lib_id "Device:C_Small") (at 124.46 66.04 0) (unit 1)
     (in_bom yes) (on_board yes) (dnp no) (fields_autoplaced)
-    (property "Reference" "C7" (at 127 64.7762 0)
+    (property "Reference" "C13" (at 127 64.7762 0)
       (effects (font (size 1.27 1.27)) (justify left))
     )
@@
       (effects (font (size 1.27 1.27)) (justify left))
     )
-    (property "Footprint" "Capacitor_SMD:C_1206_3216Metric_Pad1.33x1.80mm_HandSolder" (at 124.46 66.04 0)
+    (property "Footprint" "Capacitor_SMD:C_0805_2012Metric_Pad1.18x1.45mm_HandSolder" (at 124.46 66.04 0)
       (effects (font (size 1.27 1.27)) hide)
     )
@@
       (project "combat_2.0"
         (path "/518cdd36-e3d2-496e-a534-90a14dea15b3/75a6c3bc-fc0f-431f-8cec-1b3bc24c24b9"
-          (reference "C7") (unit 1)
+          (reference "C13") (unit 1)
         )
       )
@@
   (symbol (lib_id "Connector:Conn_01x03_Pin") (at 147.32 53.34 180) (unit 1)
     (in_bom yes) (on_board yes) (dnp no) (fields_autoplaced)
-    (property "Reference" "J10" (at 146.685 59.69 0)
+    (property "Reference" "J5" (at 146.685 59.69 0)
       (effects (font (size 1.27 1.27)))
     )
@@
       (effects (font (size 1.27 1.27)))
     )
-    (property "Footprint" "Connector_JST:JST_GH_SM02B-GHS-TB_1x02-1MP_P1.25mm_Horizontal" (at 147.32 53.34 0)
+    (property "Footprint" "Connector_Molex:Molex_PicoBlade_53398-0271_1x02-1MP_P1.25mm_Vertical" (at 147.32 53.34 0)
       (effects (font (size 1.27 1.27)) hide)
     )
@@
       (project "combat_2.0"
         (path "/518cdd36-e3d2-496e-a534-90a14dea15b3/75a6c3bc-fc0f-431f-8cec-1b3bc24c24b9"
-          (reference "J10") (unit 1)
+          (reference "J5") (unit 1)
         )
       )
@@
   (symbol (lib_id "Device:C_Small") (at 124.46 53.34 0) (unit 1)
     (in_bom yes) (on_board yes) (dnp no) (fields_autoplaced)
-    (property "Reference" "C6" (at 127 52.0762 0)
+    (property "Reference" "C12" (at 127 52.0762 0)
       (effects (font (size 1.27 1.27)) (justify left))
     )
@@
       (effects (font (size 1.27 1.27)) (justify left))
     )
-    (property "Footprint" "Capacitor_SMD:C_1206_3216Metric_Pad1.33x1.80mm_HandSolder" (at 124.46 53.34 0)
+    (property "Footprint" "Capacitor_SMD:C_0805_2012Metric_Pad1.18x1.45mm_HandSolder" (at 124.46 53.34 0)
       (effects (font (size 1.27 1.27)) hide)
     )
@@
       (project "combat_2.0"
         (path "/518cdd36-e3d2-496e-a534-90a14dea15b3/75a6c3bc-fc0f-431f-8cec-1b3bc24c24b9"
-          (reference "C6") (unit 1)
+          (reference "C12") (unit 1)
         )
       )
@@
   (symbol (lib_id "Connector:Conn_01x03_Pin") (at 146.05 66.04 180) (unit 1)
     (in_bom yes) (on_board yes) (dnp no) (fields_autoplaced)
-    (property "Reference" "J11" (at 145.415 72.39 0)
+    (property "Reference" "J4" (at 145.415 72.39 0)
       (effects (font (size 1.27 1.27)))
     )
@@
       (effects (font (size 1.27 1.27)))
     )
-    (property "Footprint" "Connector_JST:JST_GH_SM02B-GHS-TB_1x02-1MP_P1.25mm_Horizontal" (at 146.05 66.04 0)
+    (property "Footprint" "Connector_Molex:Molex_PicoBlade_53398-0271_1x02-1MP_P1.25mm_Vertical" (at 146.05 66.04 0)
       (effects (font (size 1.27 1.27)) hide)
     )
@@
       (project "combat_2.0"
         (path "/518cdd36-e3d2-496e-a534-90a14dea15b3/75a6c3bc-fc0f-431f-8cec-1b3bc24c24b9"
-          (reference "J11") (unit 1)
-        )
-      )
+          (reference "J4") (unit 1)
+        )
+      )
